File: Starbie/Starbie.kicad_sch (KiCad schematic)
At the start: 7 parts, among them J1 Conn_01x04_Pin, J2 Conn_01x08_Pin, SW1 SW_Push, SW2 SW_Push, U1 XIAO-ESP32-C3-SMD, U2 DHT11

Commit message: forgot to commit this yesterday but routed the basic pcb
Parts:
- U1: footprint Sensor:Aosong_DHT11_5.5x12.0_P2.54mm -> Imported_Parts:XIAO-ESP32-C6-DIP
- U2: footprint Imported_Parts:XIAO-ESP32-C6-DIP -> Sensor:Aosong_DHT11_5.5x12.0_P2.54mm
Changed lines of the file:
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@@
 			)
 		)
-		(property "Footprint" "Imported_Parts:XIAO-ESP32-C6-DIP"
+		(property "Footprint" "Sensor:Aosong_DHT11_5.5x12.0_P2.54mm"
 			(at 95.25 113.03 0)
 			(hide yes)
@@
 			)
 		)
-		(property "Footprint" "Sensor:Aosong_DHT11_5.5x12.0_P2.54mm"
+		(property "Footprint" "Imported_Parts:XIAO-ESP32-C6-DIP"
 			(at 112.522 119.634 0)
 			(hide yes)

Commit message: add switch, LED mood lighting and battery connectors (and testpoint also) + routed everything + rounded star edges
Parts:
- added D1: LED_RKGB, LED_THT:LED_D5.0mm-4_RGB_Staggered_Pins, symbol Device:LED_RKGB
- added J3: Conn_01x02_Socket, Connector_JST:JST_PH_B2B-PH-K_1x02_P2.00mm_Vertical, symbol Connector:Conn_01x02_Socket
- added R2, R3, R4: 220, Resistor_THT:R_Axial_DIN0204_L3.6mm_D1.6mm_P7.62mm_Horizontal, symbol Device:R
- added SW3: SW_SPDT, Button_Switch_THT:SW_Slide_SPDT_Straight_CK_OS102011MS2Q, symbol Switch:SW_SPDT
- added TP1: TestPoint, TestPoint:TestPoint_THTPad_D1.5mm_Drill0.7mm, symbol Connector:TestPoint
Connections:
- net GND: now also D1.2 (K), J3.2 (Pin_2)
- net LED_R: now reaches U1.1 (D0)
- net LED_R: now also R2.1
- net LED_G: now reaches U1.7 (D6)
- net LED_G: now also R3.1
- net LED_B: now reaches U1.8 (D7)
- net LED_B: now also R4.1
- new net: D1.4 (BA), R4.2
- new net: D1.3 (GA), R3.2
- new net: D1.1 (RA), R2.2
- new net BAT_RAW: J3.1 (Pin_1), SW3.2 (B)
- new net VBAT_SW: SW3.1 (A), TP1.1
- no-connect marks 17 -> 15
Other:
- note added: "Battery Connector"
- note added: "Mood light LED"
- note added: "Switch"
- note added: "Wire Pad"

Commit message: fixing porting error in pcb + schematic, start firmware and program led functionality
Connections:
- net LED_R: now also U1.11 (D10); no longer U1.1 (D0)
Changed lines of the file:
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@@
-	)
-	(no_connect
-		(at 171.45 99.06)
 	)
 	(no_connect
@@
 	(no_connect
 		(at 140.97 74.93)
+	)
+	(no_connect
+		(at 129.54 87.63)
 	)
 	(no_connect
@@
 		)
 	)
-	(label "LED_R"
-		(at 129.54 87.63 180)
-		(effects
-			(font
-				(size 1.27 1.27)
-			)
-			(justify right bottom)
-		)
-	)
 	(label "GPIO2"
 		(at 66.04 62.23 180)
@@
 		)
 	)
+	(label "LED_R"
+		(at 171.45 99.06 0)
+		(effects
+			(font
+				(size 1.27 1.27)
+			)
+			(justify left bottom)
+		)
+	)
